File: fanmon.brd (EAGLE design)
At the start: 77.1 x 55.9 mm, 33 parts, among them IC1 PIC18F1220P, IC2 5vdc reg, K1 G6D-1A-ASI5VDC, X1 22-23-2021, X2 22-23-2021, X3 22-23-2021, X4 22-23-2021, X5 22-23-2041

Commit message: updates
Parts:
- added R6, R7: 4.7k, resistor:0204V
Connections:
- net N$5: now also R6.1
- net N$7: now also R7.2
- net VDD: now also R6.2, R7.1
Routing:
- net N$4: track 139.9 -> 108.8 mm
- net N$10: track 100.5 -> 70.2 mm
- net N$13: track 106.5 -> 132.0 mm
- net N$1: track 48.4 -> 23.7 mm
- net VSS: track 149.3 -> 172.5 mm
- net N$5: track 102.2 -> 118.3 mm
- net N$12: track 104.4 -> 115.3 mm
- net N$11: track 84.0 -> 76.8 mm
- net VDD: track 164.5 -> 170.3 mm
- net N$14: track 10.7 -> 7.43 mm
- net N$15: track 32.6 -> 30.5 mm, vias 1 -> 0
- net N$6: track 80.3 -> 82.0 mm
- net N$7: track 73.8 -> 72.1 mm
- net N$2: track 12.5 -> 11.0 mm
- net N$9: track 16.8 -> 15.5 mm
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Other:
- board size 77.1 x 55.9 mm -> 77.1 x 52.1 mm
