File: fanmon.sch (EAGLE design)
At the start: 32 parts, among them IC1 PIC18F1220P, IC2 5vdc reg, K1 G6D-1A-ASI5VDC, X1 22-23-2021, X2 22-23-2021, X3 22-23-2021, X4 22-23-2021, X5 22-23-2041

Commit message: updates
Parts:
- added R6, R7: 4.7k, resistor:R-US_0204/2V
Connections:
- net N$5: now also R6.1
- net N$7: now also R7.2
- net VDD: now also R6.2, R7.1
Other:
- note added: "Fan alarm relay"
- note added: "Fan run LED output"
- note added: "ICSP"
- note added: "Rotation sensor inputs"
- note added: "Rotation sensor power"
- note added: "power led"
Changed lines of the file:
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@@
 <?xml version="1.0" encoding="utf-8"?>
 <!DOCTYPE eagle SYSTEM "eagle.dtd">
-<eagle version="6.6.0">
+<eagle version="7.5.0">
 <drawing>
 <settings>
@@
 <part name="SV1" library="con-lstb" deviceset="MA06-1" device=""/>
 <part name="X6" library="con-phoenix-254" deviceset="MPT2" device=""/>
+<part name="R6" library="resistor" deviceset="R-US_" device="0204/2V" value="4.7k"/>
+<part name="R7" library="resistor" deviceset="R-US_" device="0204/2V" value="4.7k"/>
+<part name="VDD2" library="supply1" deviceset="VDD" device=""/>
+<part name="VDD3" library="supply1" deviceset="VDD" device=""/>
 </parts>
 <sheets>
 <sheet>
 <plain>
+<text x="106.68" y="55.88" size="1.778" layer="91">Rotation sensor inputs</text>
+<text x="-50.8" y="53.34" size="1.778" layer="91">Rotation sensor power</text>
+<text x="-12.7" y="-20.32" size="1.778" layer="91">Fan run LED output</text>
+<text x="48.26" y="-20.32" size="1.778" layer="91">Fan run LED output</text>
+<text x="106.68" y="-22.86" size="1.778" layer="91">Fan alarm relay</text>
+<text x="7.62" y="38.1" size="1.778" layer="91">power led</text>
+<text x="-40.64" y="-7.62" size="1.778" layer="91">ICSP</text>
 </plain>
 <instances>
@@
 <instance part="X6" gate="-1" x="-20.32" y="60.96" rot="R90"/>
 <instance part="X6" gate="-2" x="-40.64" y="38.1" rot="R180"/>
+<instance part="R6" gate="G$1" x="111.76" y="58.42" rot="R90"/>
+<instance part="R7" gate="G$1" x="111.76" y="43.18" rot="R90"/>
+<instance part="VDD2" gate="G$1" x="111.76" y="66.04"/>
+<instance part="VDD3" gate="G$1" x="111.76" y="35.56" rot="R180"/>
 </instances>
 <busses>
@@
 <junction x="-33.02" y="2.54"/>
 </segment>
+<segment>
+<pinref part="R6" gate="G$1" pin="2"/>
+<pinref part="VDD2" gate="G$1" pin="VDD"/>
+</segment>
+<segment>
+<pinref part="R7" gate="G$1" pin="1"/>
+<pinref part="VDD3" gate="G$1" pin="VDD"/>
+</segment>
 </net>
 <net name="VSS" class="0">
@@
 <wire x1="99.06" y1="50.8" x2="114.3" y2="50.8" width="0.1524" layer="91"/>
 <junction x="99.06" y="50.8"/>
+<pinref part="R6" gate="G$1" pin="1"/>
+<junction x="111.76" y="53.34"/>
 </segment>
 </net>
@@
 <wire x1="99.06" y1="45.72" x2="114.3" y2="45.72" width="0.1524" layer="91"/>
 <junction x="99.06" y="45.72"/>
-</segment>
-</net>
+<pinref part="R7" gate="G$1" pin="2"/>
+<junction x="111.76" y="48.26"/>
+</segment>
+</net>
